File: W48.kicad_pcb (KiCad board)
At the start: 2 copper layers, 65.1 x 65.1 mm, 17 parts, among them P1 R_Potentiometer_Trim, T1 BC847C, T2 BC847C

Commit message: layout and gnd layer
Parts:
- moved C3 45.7 mm to (114.3, 82.2), turned to 90 degrees
- moved R1 42.8 mm to (124.5, 70.2), turned to 90 degrees
- moved D1 40.8 mm to (134.6, 106.7), turned to 90 degrees
- moved R3 31.7 mm to (122.1, 81.3), turned to 180 degrees
- moved T1 24.1 mm to (115.8, 75.2), turned to -90 degrees
- moved R2 19.9 mm to (121.2, 75.5), turned to 90 degrees
- moved T2 19.3 mm to (129.5, 88.3), turned to -90 degrees
- moved D2 19.1 mm to (129.2, 81.9), turned to 90 degrees
- moved C1 16.5 mm to (125.0, 103.1), turned to 180 degrees
- moved D3 15.1 mm to (129.2, 76.3), turned to 90 degrees
- moved R4 14.9 mm to (129.5, 95.2), turned to -90 degrees
- moved MK1 12.3 mm to (151.7, 86.8), turned to 90 degrees
- moved P1 9.15 mm to (120.1, 90.7)
- moved C2 8.63 mm to (121.9, 67.6), turned to 90 degrees
Routing:
- net Net-(C1-Pad2): track 0.00 -> 90.3 mm, vias 0 -> 6
- net Net-(C1-Pad1): track 0.00 -> 46.2 mm, vias 0 -> 2
- net Net-(D3-Pad3): track 0.00 -> 37.5 mm
- net Net-(D2-Pad2): track 0.00 -> 37.1 mm
- net Net-(C2-Pad2): track 0.00 -> 35.7 mm
- net Net-(C3-Pad1): track 0.00 -> 30.5 mm, vias 0 -> 2
- net Net-(C3-Pad2): track 0.00 -> 16.2 mm
- net Net-(D2-Pad3): track 0.00 -> 13.0 mm, vias 0 -> 2
- net Net-(C2-Pad1): track 0.00 -> 10.4 mm
- added copper zone on B.Cu, net (none)

Commit message: real gnd layer
Parts:
- moved C2 2.49 mm to (121.6, 70.1)
Connections:
- net Net-(C1-Pad2) renamed /GND
Routing:
- net /GND: track 90.3 -> 6.42 mm, vias 6 -> 5
- net Net-(D1-A): track 46.2 -> 54.2 mm, vias 2 -> 0
- net Net-(MK1-+): track 35.7 -> 38.6 mm
- net Net-(T1-B): track 10.4 -> 8.06 mm
- net Net-(T2-B): track 30.5 -> 29.4 mm
- net Net-(D2-A): track 37.1 -> 36.1 mm
- net Net-(D2-K-Pad3): track 13.0 -> 12.4 mm
- added copper zone on B.Cu, net /GND
- removed copper zone on B.Cu, net (none)
